File: usb-uart.kicad_pcb (KiCad board)
At the start: 2 copper layers, 42 x 42 mm, 24 parts, among them J1 USB_B, J2 Conn_01x04_Female, SW1 SW_Push_Open, U1 CP2102N-A01-GQFN24

Commit message: updated to build (and include) a .step 3d model of the board
Parts:
- J1: footprint Connector_USB:USB_B_OST_USB-B1HSxx_Horizontal -> 3d:OST_USB-B1HSB6
- moved J1 4.87 mm to (149.2, 60.0), turned to 90 degrees
